File: shield_opencm.brd (EAGLE design)
At the start: 2 parts

Commit message: first commit
Parts:
- added E$3: (no value), pinhead:1X04
- added E$4: (no value), pinhead:1X03
- added E$5: (no value), pinhead:1X05
- added E$6: (no value), con-wago-500:W237-103
- moved E$1 18.2 mm to (41.9, 66.0), turned to 90 degrees
- moved E$2 10.2 mm to (59.7, 66.0), turned to 90 degrees
Connections:
- new net S$1: E$1.6, E$3.4
- new net S$10: E$2.10, E$5.3
- new net S$11: E$2.11, E$5.4
- new net S$12: E$2.12, E$5.5
- new net S$13: E$1.1, E$4.1
- new net S$14: E$2.18
- new net S$2: E$1.3, E$3.1
- new net S$3: E$2.5, E$3.2
- new net S$4: E$1.2, E$3.3
- new net S$5: E$2.20
- new net S$6: E$2.7, E$4.3
- new net S$7: E$2.6, E$4.2
- new net S$8: E$2.8, E$5.1
- new net S$9: E$2.9, E$5.2
Routing:
- net S$4: track 0.00 -> 152.1 mm
- net S$3: track 0.00 -> 123.8 mm
- net S$13: track 0.00 -> 52.6 mm, vias 0 -> 2
- net S$7: track 0.00 -> 11.2 mm
- net S$6: track 0.00 -> 11.2 mm
- net S$14: track 0.00 -> 10.7 mm
- net S$5: track 0.00 -> 10.7 mm
- net S$9: track 0.00 -> 10.2 mm
- net S$8: track 0.00 -> 10.2 mm
- net S$12: track 0.00 -> 10.2 mm
- net S$11: track 0.00 -> 10.2 mm
- net S$10: track 0.00 -> 10.2 mm
- net S$2: track 0.00 -> 6.35 mm
- net S$1: track 0.00 -> 6.35 mm
Other:
- board text added: "jeykeyyy"
Changed lines of the file:
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@@
 <setting verticaltext="up"/>
 </settings>
-<grid distance="50" unitdist="mil" unit="mil" style="lines" multiple="1" display="no" altdistance="5" altunitdist="mil" altunit="mil"/>
+<grid distance="50" unitdist="mil" unit="mm" style="lines" multiple="1" display="no" altdistance="5" altunitdist="mil" altunit="mm"/>
 <layers>
 <layer number="1" name="Top" color="4" fill="1" visible="yes" active="yes"/>
@@
 <board>
 <plain>
+<text x="35.56" y="90.17" size="1.778" layer="16" rot="MR270">jeykeyyy</text>
 </plain>
 <attributes>
@@
 </autorouter>
 <elements>
-<element name="E$1" library="pinhead" library_urn="urn:adsk.eagle:library:325" package="1X20" package3d_urn="urn:adsk.eagle:package:22441/2" value="" x="49.53" y="82.55" smashed="yes">
-<attribute name="NAME" x="24.0538" y="84.3788" size="1.27" layer="25" ratio="10"/>
-<attribute name="VALUE" x="24.13" y="79.375" size="1.27" layer="27"/>
-</element>
-<element name="E$2" library="pinhead" library_urn="urn:adsk.eagle:library:325" package="1X20" package3d_urn="urn:adsk.eagle:package:22441/2" value="" x="49.53" y="64.77" smashed="yes">
-<attribute name="NAME" x="24.0538" y="66.5988" size="1.27" layer="25" ratio="10"/>
-<attribute name="VALUE" x="24.13" y="61.595" size="1.27" layer="27"/>
+<element name="E$1" library="pinhead" library_urn="urn:adsk.eagle:library:325" package="1X20" package3d_urn="urn:adsk.eagle:package:22441/2" value="" x="41.91" y="66.04" smashed="yes" rot="R90">
+<attribute name="NAME" x="40.0812" y="40.5638" size="1.27" layer="25" ratio="10" rot="R90"/>
+<attribute name="VALUE" x="45.085" y="40.64" size="1.27" layer="27" rot="R90"/>
+</element>
+<element name="E$2" library="pinhead" library_urn="urn:adsk.eagle:library:325" package="1X20" package3d_urn="urn:adsk.eagle:package:22441/2" value="" x="59.69" y="66.04" smashed="yes" rot="R90">
+<attribute name="NAME" x="57.8612" y="40.5638" size="1.27" layer="25" ratio="10" rot="R90"/>
+<attribute name="VALUE" x="62.865" y="40.64" size="1.27" layer="27" rot="R90"/>
+</element>
+<element name="E$3" library="pinhead" library_urn="urn:adsk.eagle:library:325" package="1X04" package3d_urn="urn:adsk.eagle:package:22407/2" value="" x="35.56" y="50.8" smashed="yes" rot="R90">
+<attribute name="NAME" x="33.7312" y="45.6438" size="1.27" layer="25" ratio="10" rot="R90"/>
+<attribute name="VALUE" x="38.735" y="45.72" size="1.27" layer="27" rot="R90"/>
+</element>
+<element name="E$4" library="pinhead" library_urn="urn:adsk.eagle:library:325" package="1X03" package3d_urn="urn:adsk.eagle:package:22458/2" value="" x="69.85" y="52.07" smashed="yes" rot="R90">
+<attribute name="NAME" x="68.0212" y="48.1838" size="1.27" layer="25" ratio="10" rot="R90"/>
+<attribute name="VALUE" x="73.025" y="48.26" size="1.27" layer="27" rot="R90"/>
+</element>
+<element name="E$5" library="pinhead" library_urn="urn:adsk.eagle:library:325" package="1X05" package3d_urn="urn:adsk.eagle:package:22469/2" value="" x="69.85" y="64.77" smashed="yes" rot="R90">
+<attribute name="NAME" x="68.0212" y="58.3438" size="1.27" layer="25" ratio="10" rot="R90"/>
+<attribute name="VALUE" x="73.025" y="58.42" size="1.27" layer="27" rot="R90"/>
+</element>
+<element name="E$6" library="con-wago-500" library_urn="urn:adsk.eagle:library:195" package="W237-103" package3d_urn="urn:adsk.eagle:package:10691/1" value="" x="71.12" y="83.82" smashed="yes" rot="R270">
+<attribute name="NAME" x="63.6578" y="89.5058" size="1.27" layer="25" ratio="10" rot="R270"/>
+<attribute name="VALUE" x="66.1724" y="89.1248" size="1.27" layer="27" ratio="10" rot="R270"/>
 </element>
 </elements>
 <signals>
+<signal name="S$1">
+<contactref element="E$3" pad="4"/>
+<contactref element="E$1" pad="6"/>
+<wire x1="35.56" y1="54.61" x2="41.91" y2="54.61" width="0.508" layer="16"/>
+</signal>
+<signal name="S$2">
+<contactref element="E$3" pad="1"/>
+<contactref element="E$1" pad="3"/>
+<wire x1="35.56" y1="46.99" x2="41.91" y2="46.99" width="0.508" layer="16"/>
+</signal>
+<signal name="S$3">
+<contactref element="E$3" pad="2"/>
+<wire x1="35.56" y1="49.53" x2="29.21" y2="49.53" width="0.508" layer="16"/>
+<wire x1="29.21" y1="49.53" x2="27.94" y2="50.8" width="0.508" layer="16"/>
+<wire x1="27.94" y1="50.8" x2="27.94" y2="92.71" width="0.508" layer="16"/>
+<wire x1="27.94" y1="92.71" x2="30.48" y2="95.25" width="0.508" layer="16"/>
+<wire x1="30.48" y1="95.25" x2="50.8" y2="95.25" width="0.508" layer="16"/>
+<wire x1="50.8" y1="95.25" x2="54.61" y2="91.44" width="0.508" layer="16"/>
+<wire x1="54.61" y1="91.44" x2="54.61" y2="52.07" width="0.508" layer="16"/>
+<contactref element="E$2" pad="5"/>
+<wire x1="54.61" y1="52.07" x2="59.69" y2="52.07" width="0.508" layer="16"/>
+</signal>
+<signal name="S$4">
+<contactref element="E$3" pad="3"/>
+<wire x1="35.56" y1="52.07" x2="33.02" y2="52.07" width="0.508" layer="16"/>
+<wire x1="33.02" y1="52.07" x2="31.75" y2="53.34" width="0.508" layer="16"/>
+<wire x1="31.75" y1="53.34" x2="31.75" y2="90.17" width="0.508" layer="16"/>
+<wire x1="31.75" y1="90.17" x2="34.29" y2="92.71" width="0.508" layer="16"/>
+<wire x1="34.29" y1="92.71" x2="49.53" y2="92.71" width="0.508" layer="16"/>
+<wire x1="49.53" y1="92.71" x2="52.07" y2="90.17" width="0.508" layer="16"/>
+<wire x1="52.07" y1="90.17" x2="52.07" y2="38.1" width="0.508" layer="16"/>
+<wire x1="52.07" y1="38.1" x2="49.53" y2="35.56" width="0.508" layer="16"/>
+<wire x1="49.53" y1="35.56" x2="35.56" y2="35.56" width="0.508" layer="16"/>
+<wire x1="35.56" y1="35.56" x2="33.02" y2="38.1" width="0.508" layer="16"/>
+<wire x1="33.02" y1="38.1" x2="33.02" y2="44.45" width="0.508" layer="16"/>
+<contactref element="E$1" pad="2"/>
+<wire x1="33.02" y1="44.45" x2="41.91" y2="44.45" width="0.508" layer="16"/>
+</signal>
+<signal name="S$13">
+<contactref element="E$1" pad="1"/>
+<wire x1="41.91" y1="41.91" x2="41.91" y2="38.1" width="0.508" layer="16"/>
+<via x="41.91" y="38.1" extent="1-16" drill="1" diameter="1.3" shape="square"/>
+<wire x1="41.91" y1="38.1" x2="41.91" y2="33.02" width="0.508" layer="1"/>
+<via x="41.91" y="33.02" extent="1-16" drill="1" diameter="1.3" shape="square"/>
+<wire x1="41.91" y1="33.02" x2="68.58" y2="33.02" width="0.508" layer="16"/>
+<wire x1="68.58" y1="33.02" x2="69.85" y2="34.29" width="0.508" layer="16"/>
+<contactref element="E$4" pad="1"/>
+<wire x1="69.85" y1="34.29" x2="69.85" y2="49.53" width="0.508" layer="16"/>
+</signal>
+<signal name="S$6">
+<contactref element="E$2" pad="7"/>
+<wire x1="59.69" y1="57.15" x2="63.5" y2="57.15" width="0.508" layer="16"/>
+<wire x1="63.5" y1="57.15" x2="66.04" y2="54.61" width="0.508" layer="16"/>
+<contactref element="E$4" pad="3"/>
+<wire x1="66.04" y1="54.61" x2="69.85" y2="54.61" width="0.508" layer="16"/>
+</signal>
+<signal name="S$7">
+<contactref element="E$2" pad="6"/>
+<wire x1="59.69" y1="54.61" x2="62.23" y2="54.61" width="0.508" layer="16"/>
+<wire x1="62.23" y1="54.61" x2="64.77" y2="52.07" width="0.508" layer="16"/>
+<contactref element="E$4" pad="2"/>
+<wire x1="64.77" y1="52.07" x2="69.85" y2="52.07" width="0.508" layer="16"/>
+</signal>
+<signal name="S$8">
+<contactref element="E$2" pad="8"/>
+<contactref element="E$5" pad="1"/>
+<wire x1="59.69" y1="59.69" x2="68.58" y2="59.69" width="0.508" layer="16"/>
+<wire x1="68.58" y1="59.69" x2="69.85" y2="59.69" width="0.508" layer="16"/>
+</signal>
+<signal name="S$9">
+<contactref element="E$2" pad="9"/>
+<contactref element="E$5" pad="2"/>
+<wire x1="59.69" y1="62.23" x2="69.85" y2="62.23" width="0.508" layer="16"/>
+</signal>
+<signal name="S$10">
+<contactref element="E$2" pad="10"/>
+<contactref element="E$5" pad="3"/>
+<wire x1="59.69" y1="64.77" x2="69.85" y2="64.77" width="0.508" layer="16"/>
+</signal>
+<signal name="S$11">
+<contactref element="E$2" pad="11"/>
+<contactref element="E$5" pad="4"/>
+<wire x1="59.69" y1="67.31" x2="69.85" y2="67.31" width="0.508" layer="16"/>
+</signal>
+<signal name="S$12">
+<contactref element="E$2" pad="12"/>
+<contactref element="E$5" pad="5"/>
+<wire x1="59.69" y1="69.85" x2="69.85" y2="69.85" width="0.508" layer="16"/>
+</signal>
+<signal name="S$5">
+<contactref element="E$2" pad="20"/>
+<wire x1="59.69" y1="90.17" x2="63.5" y2="90.17" width="1.016" layer="16"/>
+<wire x1="63.5" y1="90.17" x2="64.77" y2="88.9" width="1.016" layer="16"/>
+<wire x1="64.77" y1="88.9" x2="69.85" y2="88.9" width="1.016" layer="16"/>
+</signal>
+<signal name="S$14">
+<contactref element="E$2" pad="18"/>
+<wire x1="59.69" y1="85.09" x2="62.23" y2="85.09" width="1.016" layer="16"/>
+<wire x1="62.23" y1="85.09" x2="63.5" y2="83.82" width="1.016" layer="16"/>
+<wire x1="63.5" y1="83.82" x2="69.85" y2="83.82" width="1.016" layer="16"/>
+</signal>
 </signals>
 <mfgpreviewcolors>
